File: hardware/REV2/Board1/HR_Avionics_REV2_Board1.kicad_pcb (KiCad board)
At the start: 2 copper layers, 100 x 50 mm, 150 parts, among them J1 Conn_01x02_Socket, J10 Conn_01x02_Socket, J11 Conn_01x02_Socket, J12 Conn_01x03_Socket, J2 Conn_01x02_Socket, J3 Conn_01x02_Socket, J4 Conn_01x02_Socket, J5 Conn_01x02_Socket, J6 Conn_01x02_Socket, J7 Conn_01x06_Socket, J8 Conn_01x02_Socket, J9 Conn_01x03_Socket, Q1 TJ60S04M3L(T6L,1NQ, Q10 TJ60S04M3L(T6L,1NQ, Q11 BSS138, Q12 BSS138, Q13 BSS138, Q2 TJ60S04M3L(T6L,1NQ, Q3 TJ60S04M3L(T6L,1NQ, Q4 TJ60S04M3L(T6L,1NQ, Q5 MTB7D0N06RJ3, Q6 MTB7D0N06RJ3, Q7 MTB7D0N06RJ3, Q8 MTB7D0N06RJ3, Q9 TJ60S04M3L(T6L,1NQ, U1 LTC4353, U16 USBLC6-4SC6, U18 TCAN3414DR, U2 AZ1117CH-3.3TRG1, U3 MCP1402T-E_OT, U4 STM32F303K8Tx, U5 SSM6J808RLF, U6 SSM6J808RLF, U7 INA219AIDR, U8 LMR51635, U9 MCP1402T-E_OT, Y2 CSTNE16M0V530000R0

Commit message: Update PCB
Parts:
- C13, C14, C15, C16, C17, C18, C20, D10, D16, D17, FB3, FL1, R13, R17, R23, R26, R28, R29, R30, R31, R32, R34, U18, U4, Y2: moved to B.Cu
- moved R17 147.3 mm to (195.3, 64.3), turned to -90 degrees
- moved R26 146.5 mm to (193.8, 64.3), turned to 90 degrees
- moved R13 143.7 mm to (192.0, 64.3), turned to -90 degrees
- moved R23 142.8 mm to (190.4, 64.3), turned to 90 degrees
- moved U4 133.4 mm to (198.8, 72.0)
- moved Y2 121.5 mm to (191.3, 73.7), turned to -90 degrees
- moved C20 120.2 mm to (212.3, 92.1), turned to 90 degrees
- moved C15 118.9 mm to (193.3, 78.6), turned to 90 degrees
- moved Q6 116.6 mm to (174.8, 92.4)
- moved C13 115.6 mm to (206.4, 67.4), turned to 180 degrees
- moved Q5 113.8 mm to (174.9, 65.8)
- moved Q1 112.8 mm to (171.8, 56.9), turned to -90 degrees
- moved J9 112.3 mm to (204.7, 87.2)
- moved J12 111.4 mm to (215.7, 87.2)
- moved Q3 110.1 mm to (168.1, 77.3), turned to 90 degrees
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Connections:
- FL1 pad 1: Net-(U18-CANL) -> Net-(U18-CANH)
- FL1 pad 2: Net-(J12-Pin_2) -> Net-(J12-Pin_1)
- FL1 pad 3: Net-(J12-Pin_1) -> Net-(J12-Pin_2)
- FL1 pad 4: Net-(U18-CANH) -> Net-(U18-CANL)

Commit message: Update PCB
Parts:
- removed R53: 0, Resistor_SMD:R_0603_1608Metric_Pad0.98x0.95mm_HandSolder
- added J15: S2711-46R, pq_k_gentaro:S2711-46R, B.Cu at (178.7, 68.9)
- added J16: S2711-46R, pq_k_gentaro:S2711-46R, B.Cu at (189.8, 53.9)
- added J17: S2711-46R, pq_k_gentaro:S2711-46R, B.Cu at (192.3, 83.8)
- added J18: S2711-46R, pq_k_gentaro:S2711-46R, B.Cu at (208.7, 69.5)
- added U10: S01-30300500, Unknown:S01-30300500, B.Cu at (193.5, 70.1)
- C2, C21, C22, C23, C24, C25, C26, C3, C39, C40, C41, C42, C43, C44, C60, D15, D18, D3, D4, D5, D6, D8, D9, F1, F2, L1, Q7, Q8, R27, R3, R33, R4, R5, R52, U2, U3, U8, U9: moved to B.Cu
- moved R27 171.0 mm to (220.1, 83.0), turned to 90 degrees
- moved R33 164.2 mm to (213.0, 80.9), turned to 180 degrees
- moved C21 161.0 mm to (227.4, 65.1), turned to 180 degrees
- moved Q7 155.7 mm to (225.9, 73.5), turned to 90 degrees
- moved D18 154.2 mm to (228.5, 51.2), turned to 90 degrees
- moved D11 153.2 mm to (236.9, 92.3), turned to 180 degrees
- moved C26 152.2 mm to (217.7, 65.1), turned to 180 degrees
- moved C19 149.1 mm to (210.6, 146.4)
- moved D9 144.3 mm to (227.9, 88.7), turned to 90 degrees
- moved Q8 143.1 mm to (214.6, 73.6), turned to 90 degrees
- moved D5 141.4 mm to (223.8, 51.2), turned to 90 degrees
- moved Q10 137.4 mm to (188.5, 142.6)
- moved Q9 137.4 mm to (188.5, 134.4)
- moved D3 136.0 mm to (219.0, 51.2), turned to 90 degrees
- moved D4 134.8 mm to (225.8, 59.7), turned to 180 degrees
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Connections:
- C21 pad 1: Net-(D18-A2) -> Net-(D18-A1)
- C26 pad 1: Net-(D3-A2) -> Net-(D3-A1)
- D18 pad 1: GNDPWR -> Net-(D18-A1)
- D18 pad 2: Net-(D18-A2) -> GNDPWR
- D3 pad 1: GNDPWR -> Net-(D3-A1)
- D3 pad 2: Net-(D3-A2) -> GNDPWR
- D4 pad 1: Net-(D18-A2) -> Net-(D18-A1)
- D5 pad 1: GNDPWR -> Net-(D4-A)
- D5 pad 2: Net-(D4-A) -> GNDPWR
- D6 pad 1: GNDPWR -> Net-(D6-A1)
- D6 pad 2: Net-(D6-A2) -> GNDPWR
- D8 pad 1: Net-(D3-A2) -> Net-(D3-A1)
- D8 pad 2: Net-(D6-A2) -> Net-(D6-A1)
- F1 pad 1: Net-(D18-A2) -> Net-(D18-A1)
- F2 pad 1: Net-(D3-A2) -> Net-(D3-A1)
- J3 pad 1: Net-(D18-A2) -> Net-(D18-A1)
- J4 pad 1: Net-(D3-A2) -> Net-(D3-A1)
- J4 pad 2: Net-(D6-A2) -> Net-(D6-A1)
- Q8 pad 2: Net-(D6-A2) -> Net-(D6-A1)
- U8 pad 2: Net-(U8-EN) -> VDC
Other:
- copper layers 2 -> 4

Commit message: Update PCB
Parts:
- F3, F5, F6: footprint Capacitor_SMD:C_1210_3225Metric_Pad1.33x2.70mm_HandSolder -> Fuse:Fuse_1210_3225Metric_Pad1.42x2.65mm_HandSolder
- U16: moved to B.Cu
- moved U6 168.9 mm to (220.5, 65.5), turned to -90 degrees
- moved U5 159.7 mm to (212.3, 65.5), turned to -90 degrees
- moved C10 143.3 mm to (217.2, 65.6), turned to 90 degrees
- moved C12 133.0 mm to (184.8, 54.0), turned to 180 degrees
- moved C27 126.9 mm to (181.5, 89.8)
- moved R9 121.4 mm to (192.9, 72.3)
- moved R25 114.8 mm to (216.5, 62.8)
- moved R24 112.6 mm to (215.3, 65.8), turned to 90 degrees
- moved C5 110.5 mm to (201.5, 57.9), turned to -90 degrees
- moved C11 107.0 mm to (226.4, 64.4), turned to 90 degrees
- moved U16 105.4 mm to (202.9, 58.4)
- moved F6 103.0 mm to (232.7, 64.4), turned to 180 degrees
- moved F5 102.9 mm to (232.7, 61.1), turned to 180 degrees
- moved F3 102.6 mm to (232.7, 67.7), turned to 180 degrees
- moved C6 102.6 mm to (193.7, 64.5)
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Routing:
- net Net-(D2-A): track 0.00 -> 49.0 mm
- net VEX: track 0.00 -> 25.5 mm
- net Net-(Q5-G): track 0.00 -> 22.6 mm
- net Net-(D1-A): track 0.00 -> 19.3 mm
- net Net-(Q6-G): track 0.00 -> 18.3 mm
- net Net-(D1-K): track 0.00 -> 17.4 mm
- net Net-(Q5-D): track 0.00 -> 15.8 mm
- net Net-(U7-IN+): track 0.00 -> 11.3 mm
- net Net-(U7-IN-): track 0.00 -> 10.7 mm
- net Net-(S1-COM): track 0.00 -> 7.84 mm
- net Net-(S3-COM): track 0.00 -> 7.46 mm
- net Net-(U1-CPO1): track 0.00 -> 5.68 mm
- net Net-(U1-CPO2): track 0.00 -> 5.29 mm
- net VDC: track 0.00 -> 4.54 mm
- net Net-(U1-VCC): track 0.00 -> 3.34 mm
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- added copper zone on F.Cu, net 3.3V
- added copper zone on In1.Cu, net GNDPWR
- added copper zone on In2.Cu, net GNDPWR
- added copper zone on F.Cu, net Net-(D1-A)
- added copper zone on F.Cu, net Net-(D1-K)
- added copper zone on F.Cu, net Net-(D16-A2)
- added copper zone on F.Cu, net Net-(D17-A2)
- added copper zone on F.Cu, net Net-(D2-K)
- added copper zone on F.Cu, net Net-(Q5-D)
- added copper zone on F.Cu, net Net-(U1-~{EN1})
- added copper zone on F.Cu, net Net-(U1-~{EN2})
- added copper zone on F.Cu, net Net-(U1-~{ONST1})
- added copper zone on F.Cu, net Net-(U1-~{ONST2})
- added copper zone on F.Cu, net VBATT
- added copper zone on F.Cu, net VDC
- added copper zone on F.Cu, net VEX
