File: hardware/REV2/Board2/HR_Avionics_REV2_Board2.kicad_sch (KiCad schematic)
At the start: 14 parts, among them J12 Conn_01x03_Socket, J9 Conn_01x03_Socket, U1 LSM6DSK320XTR, U18 TCAN3414DR, U2 BMP585, U3 STM32H523RETx, U4 MAX-M10S, U5 E22-900T30D_E220-900T22S(JP)_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, U6 E22-900T30D_E220-900T22S(JP)_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

Commit message: Update sch and pcb
Parts:
- removed R34: 120, Resistor_SMD:R_0603_1608Metric_Pad0.98x0.95mm_HandSolder, symbol Device:R
- added C1: 16SEPF1000M, Capacitor_THT:CP_Radial_D10.0mm_P5.00mm, symbol Device:C_Polarized_Small
- added C17, C18, C21, C24, C25, C26, C27, C28, C29, C30, C31, C32, C33, C34, C36, C37, C38, C41, C42, C43, C44, C45, C47, C49, C50, C51, C52, C53: 0.1u, Capacitor_SMD:C_0603_1608Metric_Pad1.08x0.95mm_HandSolder, symbol Device:C_Small
- added C2, C3: 16SKV100M6.3X5.5, Capacitor_SMD:CP_Elec_6.3x5.4, symbol Device:C_Polarized_Small
- added C22, C23, C35, C48: 1u, Capacitor_SMD:C_0603_1608Metric_Pad1.08x0.95mm_HandSolder, symbol Device:C_Small
- added C39, C40: 2.2u, Capacitor_SMD:C_0603_1608Metric_Pad1.08x0.95mm_HandSolder, symbol Device:C_Small
- added C46: 4.7u, Capacitor_SMD:C_0805_2012Metric_Pad1.18x1.45mm_HandSolder, symbol Device:C_Small
- added C7, C8: 4.7u, Capacitor_SMD:C_1210_3225Metric_Pad1.33x2.70mm_HandSolder, symbol Device:C_Small
- added C9: 3.3u, Capacitor_SMD:C_1210_3225Metric_Pad1.33x2.70mm_HandSolder, symbol Device:C_Small
- added D11: SMBJ16CA(576-SMBJ16CA), Diode_SMD:D_SMB, symbol Device:D_TVS_Small
- added D13: MA10EB045, Diode_SMD:D_SOD-123, symbol Device:D_Schottky_Small
- added D15, D16: D_Schottky_Small, Diode_SMD:D_SOD-123, symbol Device:D_Schottky_Small
- added F2: 1210L300SLWR, Fuse:Fuse_1210_3225Metric_Pad1.42x2.65mm_HandSolder, symbol Device:Polyfuse_Small
- added FB1: MI0805K601R-10, Inductor_SMD:L_0805_2012Metric_Pad1.05x1.20mm_HandSolder, symbol Device:FerriteBead_Small
- added FB3: 782639601, Inductor_SMD:L_0603_1608Metric_Pad1.05x0.95mm_HandSolder, symbol Device:FerriteBead_Small
- added H1, H2, H3, H4: MountingHole_Pad, MountingHole:MountingHole_3.2mm_M3_ISO7380_Pad, symbol Mechanical:MountingHole_Pad
- added IC2, IC3: XC8114AA01PR-G, Unknown:XC6901D901PRG, symbol Unknown:XC8114AA01PR-G
- added J1: 5077CR-16SMC2-BK-TR, Unknown:NELTRON_5077CR-16SMC2-BK-TR, symbol Unknown:5077CR-16SMC2-BK-TR
- added J10: Conn_01x06_Pin, Connector_JST:JST_XH_B6B-XH-A_1x06_P2.50mm_Vertical, symbol Connector:Conn_01x06_Pin
- added J15, J16, J17, J18: S2711-46R, pq_k_gentaro:S2711-46R, symbol Connector_Generic:Conn_01x01
- added J5, J7: Conn_01x02_Socket, Connector_JST:JST_XH_S2B-XH-A_1x02_P2.50mm_Horizontal, symbol Connector:Conn_01x02_Socket
- added J6: Conn_01x02_Socket, Connector_JST:JST_VH_B2PS-VH_1x02_P3.96mm_Horizontal, symbol Connector:Conn_01x02_Socket
- added L1: BLM18PG471SN1D, Inductor_SMD:L_0603_1608Metric_Pad1.05x0.95mm_HandSolder, symbol Device:L_Ferrite
- added Q1: TJ60S04M3L(T6L,1NQ, Package_TO_SOT_SMD:TO-252-2, symbol Simulation_SPICE:PMOS
- added Q8: BSS138, Package_TO_SOT_SMD:SOT-23, symbol Transistor_FET:BSS138
- added R1: 0, Resistor_SMD:R_0603_1608Metric_Pad0.98x0.95mm_HandSolder, symbol Device:R_Small
- added R10, R11, R14, R3, R5, R7: 47k, Resistor_SMD:R_0603_1608Metric_Pad0.98x0.95mm_HandSolder, symbol Device:R_Small
- added R12, R16, R4, R8, R9: 1k, Resistor_SMD:R_0603_1608Metric_Pad0.98x0.95mm_HandSolder, symbol Device:R_Small
- added R13, R15: 10k, Resistor_SMD:R_0603_1608Metric_Pad0.98x0.95mm_HandSolder, symbol Device:R_Small
- added R17, R18: 5.1k, Resistor_SMD:R_0603_1608Metric_Pad0.98x0.95mm_HandSolder, symbol Device:R_Small
- added R2: 100, Resistor_SMD:R_0603_1608Metric_Pad0.98x0.95mm_HandSolder, symbol Device:R_Small
- added R6: 120, Resistor_SMD:R_0603_1608Metric_Pad0.98x0.95mm_HandSolder, symbol Device:R_Small
- added S3, S4: SS12SDP2, Unknown:SS12SDP2, symbol Unknown:SS12SDP2
- added SW1: PTS645SK50SMTR92LFS, Unknown:SW4_PTS645SK50SMTR92LFS_CNK, symbol Unknown:PTS645SK50SMTR92LFS
- added U10: ASGPDF254.A, Unknown:ASGPDF254.A, symbol Unknown:ASGPDF254.A
- added U11: M78AR05-1/M78AR033-1, Unknown:M78AR05-1_M78AR033-1, symbol Unknown:M78AR05-1/M78AR033-1
- added U12: UGCM1205XP, Unknown:UGCM1205XP, symbol Unknown:UGCM1205XP
- added U13: ADP151AUJZ-3.3, Package_TO_SOT_SMD:TSOT-23-5, symbol Unknown:ADP151AUJZ-3.3
- added U14: BME280, Package_LGA:Bosch_LGA-8_2.5x2.5mm_P0.65mm_ClockwisePinNumbering, symbol Sensor:BME280
- added U15: S01-30300500, Unknown:S01-30300500, symbol Unknown:S01-30300500
- added U16: FT230XS, Package_SO:SSOP-16_3.9x4.9mm_P0.635mm, symbol Interface_USB:FT230XS
- added U17: USBLC6-2SC6, Package_TO_SOT_SMD:SOT-23-6, symbol Power_Protection:USBLC6-2SC6
- added U19: USBLC6-4SC6, Package_TO_SOT_SMD:SOT-23-6, symbol Power_Protection:USBLC6-4SC6
- added U20, U21, U7: MB85RS4MTYPF-G-BCERE1, Package_SO:SOIC-8_5.3x5.3mm_P1.27mm, symbol Unknown:MB85RS4MTYPF-G-BCERE1
- added U8, U9: TC7S14F, Package_TO_SOT_SMD:TSOT-23-5_HandSoldering, symbol 74xGxx:74LVC1G14
Connections:
- net GND: now reaches U4.1 (GND), U4.10 (GND), U4.12 (GND)
- net GND: now also U1.2 (SDx), U1.3 (SCx), U1.6 (GND), U1.7 (GND), U2.6 (VSS), U3.12 (VSSA), U3.18 (VSS), U3.31 (VSS), U3.47 (VSS), U3.63 (VSS), U5.10 (GND), U5.11 (GND), U5.7 (GND), U5.8 (GND), U5.9 (GND), U6.10 (GND), U6.11 (GND), U6.7 (GND), U6.8 (GND), U6.9 (GND), C1.2, C17.1, C18.1, C2.2, C21.1, C22.1, C23.1, C24.1, C25.2, C26.2, C27.2, C28.2, C29.2, C3.2, C30.2, C31.2, C32.2, C33.2, C34.2, C35.2, C36.2, C37.1, C38.1, C39.2, C40.2, C41.1, C42.1, C43.1, C44.1, C45.1, C46.1, C47.1, C48.1, C49.1, C50.1, C51.1, C52.2, C53.2, C7.2, C8.2, C9.2, D11.1 (A1), IC2.1 (VSS), IC2.2 (EP_1), IC2.6 (EP_2), IC2.7 (EP_3), IC3.1 (VSS), IC3.2 (EP_1), IC3.6 (EP_2), IC3.7 (EP_3), J1.A1_B12 (GND), J1.B1_A12 (GND), J1.S1 (SHIELD), J1.S2 (SHIELD), J1.S3 (SHIELD), J1.S4 (SHIELD), J10.3 (Pin_3), J5.2 (Pin_2), J6.2 (Pin_2), J7.2 (Pin_2), Q8.2 (S), R17.1, R18.1, R5.2, S3.1 (NC), S4.1 (NC), SW1.3, SW1.4, U10.2 (GND), U10.3 (GND), U10.4 (GND), U10.5 (GND), U10.6 (GND), U10.7 (GND), U10.8 (GND), U10.9 (GND), U11.2 (GND), U13.2 (GND), U14.1 (GND), U14.7 (GND), U16.13 (GND), U16.5 (GND), U17.2 (GND), U19.2 (GND), U20.4 (VSS), U21.4 (VSS), U7.4 (VSS), U8.3 (GND), U9.3 (GND)
- net at U4.11 (RF_IN): now also L1.2, U10.1 (ANT)
- net at U4.14 (VCC_RF): now also R2.1
- net UART4_MISO: now reaches U4.2 (TXD)
- net UART4_MISO: now also U16.1 (TXD)
- net UART4_MOSI: now reaches U4.3 (RXD)
- net UART4_MOSI: now also U16.4 (RXD)
- net GNSS_TIMEPULSE: now reaches U4.4 (TIMEPULSE)
- net at U4.5 (EXTINT): now also R1.2
- net +3.3V_GNSS: now reaches U4.6 (V_BCKP)
- net +3.3V_GNSS: now also U4.7 (VCC_IO), U4.8 (VCC), C23.2, C25.1, C26.1, D16.2 (A), R7.1, U13.5 (VOUT)
- net ~{GNSS_RESET}: now reaches U4.9 (~{RESET})
- net ~{GNSS_RESET}: now also R7.2
- net at D10.1 (K), FL1.3, J12.2 (Pin_2)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: now also R6.2
- net LORA1_M0: now reaches U5.1 (M0)
- net LORA1_M1: now reaches U5.2 (M1)
- net USART1_MOSI: now reaches U5.3 (RXD)
- net USART1_MISO: now reaches U5.4 (TXD)
- net LORA1_AUX: now reaches U5.5 (AUX)
- net +5V: now reaches U5.6 (VCC)
- net +5V: now also U6.6 (VCC), C2.1, C21.2, C22.2, C3.1, C34.1, C35.1, C36.1, C49.2, C8.1, D13.1 (K), D15.1 (K), D16.1 (K), IC2.5 (VOUT), IC3.5 (VOUT), U11.1 (VIN), U12.1 (VIN), U13.1 (VIN), U13.3 (EN)
- net SPI2_SCK: now reaches U2.1 (SCX)
- net SPI2_MOSI: now reaches U2.2 (SDX)
- net SPI2_MISO: now reaches U2.3 (SDO)
- net +3.3V: now reaches U2.4 (VDDIO)
- net +3.3V: now also U1.5 (VDDIO), U1.8 (VDD), U2.8 (VDD), U3.1 (VBAT), U3.19 (VDD), U3.32 (VDD), U3.48 (VDD), U3.64 (VDD), C27.1, C28.1, C29.1, C30.1, C31.1, C32.1, C33.1, C41.2, C42.2, C43.2, C44.2, C45.2, C46.2, C52.1, C53.1, C9.1, D15.2 (A), FB3.1, J10.1 (Pin_1), R10.2, R11.2, R14.2, S4.3 (NO), U11.3 (VOUT), U14.6 (VDDIO), U14.8 (VDD), U19.5 (VBUS), U20.8 (VDD), U21.8 (VDD), U7.8 (VDD), U8.5 (VCC), U9.5 (VCC)
- net BMP585_INT: now reaches U2.5 (INT)
- net ~{SPI2_CS}: now reaches U2.7 (CSB)
- net at U3.13 (VDDA): now also C47.2, C48.2, FB3.2
- net at U3.30 (VCAP): now also C40.1
- net at U3.60 (BOOT0): now also R13.2
- net at U3.62 (VCAP): now also C39.1
- net at U3.7 (NRST): now also R15.1
- net LORA2_M0: now reaches U6.1 (M0)
- net LORA2_M1: now reaches U6.2 (M1)
- net USART2_MOSI: now reaches U6.3 (RXD)
- net USART2_MISO: now reaches U6.4 (TXD)
- net LORA2_AUX: now reaches U6.5 (AUX)
- net at S2.2 (COM): now also R6.1
- net SPI1_MISO: now reaches U1.1 (SDO/TA0)
- net ~{SPI1_CS}: now reaches U1.12 (CS)
- net SPI1_SCK: now reaches U1.13 (SCL)
- net SPI1_MOSI: now reaches U1.14 (SDA)
- net LSM_INT1: now reaches U1.4 (INT1)
- net LSM_INT2: now reaches U1.9 (INT2)
- new net: F2.2, FB1.1, U17.5 (VBUS)
- new net: Q1.1 (G), R3.2, R8.1
- new net: R8.2, S3.2 (COM)
- new net: J1.A5 (CC1), R18.2
- new net: C1.1, C17.2, C7.1, IC2.3 (EN), IC2.4 (VIN), Q1.2 (D)
- new net: D11.2 (A2), J6.1 (Pin_1), Q1.3 (S), R3.1
- new net: D13.2 (A), Q8.3 (D), U12.2 (GND)
- new net: R16.1, U16.11 (~{RESET})
- new net: C50.2, R16.2, U16.10 (3V3OUT), U16.3 (VCCIO)
- new net: J7.1 (Pin_1), R11.1, R12.1
- new net: J1.B5 (CC2), R17.2
- new net: C38.2, R12.2, U9.2
- new net: J5.1 (Pin_1), R10.1, R9.1
- new net: C37.2, R9.2, U8.2
- new net: F2.1, J1.A4_B9 (VBUS), J1.B4_A9 (VBUS)
- new net: J1.A6 (DP1), J1.B6 (DP2), U17.1 (I/O1)
- new net: J1.A7 (DN1), J1.B7 (DN2), U17.3 (I/O2)
- new net: Q8.1 (G), R4.2, R5.1
- new net: C24.2, L1.1, R2.2
- new net: R13.1, S4.2 (COM)
- new net: U16.9 (USBDM), U17.4 (I/O2)
- new net: U16.8 (USBDP), U17.6 (I/O1)
- new net BUZZER_EN: R4.1
- new net FLIGHT_PIN1: U8.4, U9.4
- new net GNDPWR: H1.1, H2.1, H3.1, H4.1, J15.1 (Pin_1), J16.1 (Pin_1), J17.1 (Pin_1), J18.1 (Pin_1)
- new net GNSS_EXTINT: R1.1
- new net SPI3_MISO: U14.5 (SDO)
- new net SPI3_MOSI: U14.3 (SDI)
- new net SPI3_SCK: U14.4 (SCK)
- new net SPI4_MISO: U20.2 (SO), U21.2 (SO), U7.2 (SO)
- new net SPI4_MOSI: U20.5 (SI), U21.5 (SI), U7.5 (SI)
- new net SPI4_SCK: U20.6 (SCK), U21.6 (SCK), U7.6 (SCK)
- new net SWCLK: J10.2 (Pin_2), U19.1 (I/O1)
- new net SWDIO: J10.4 (Pin_4), U19.3 (I/O2)
- new net SWO: J10.6 (Pin_6), U19.6 (I/O4)
- new net VBUS: C18.2, C51.2, FB1.2, IC3.3 (EN), IC3.4 (VIN), U16.12 (VCC)
- new net ~{FRAM1_CS}: U7.1 (~{CS})
- new net ~{FRAM1_WP}: U7.3 (~{WP})
- new net ~{FRAM2_CS}: U20.1 (~{CS})
- new net ~{FRAM2_WP}: U20.3 (~{WP})
- new net ~{FRAM3_CS}: U21.1 (~{CS})
- new net ~{FRAM3_WP}: U21.3 (~{WP})
- new net ~{NRST}: J10.5 (Pin_5), R14.1, R15.2, SW1.1, SW1.2, U19.4 (I/O3)
- new net ~{SPI3_CS}: U14.2 (CSB)
- no-connect marks 1 -> 22
Other:
- note added: "S2711-46R"
- moved on the sheet: C20, D10, FL1, J12, J9, S2, U1, U18, U2, U3, U4, U5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

Commit message: Update sch
Other:
- note added: "5V以上は印加しない"
- note added: "IC3はUSB給電時用でソフトスタート機能も兼ねる IC2とIC3で理想ダイオードOR．"
- note added: "LED"
- note added: "MCU"
- note added: "USB"
- note added: "ねじ穴・シールド"
- note added: "センサ"
- note added: "フライトピン"
- note added: "ブザー"
- note added: "記憶装置"
- note added: "通信"
- note added: "電源回路"
- moved on the sheet: C1, C17, C18, C2, C20, C21, C22, C23, C24, C25, C26, C27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
