File: hardware/REV2/Board2/HR_Avionics_REV2_Board2.kicad_pcb (KiCad board)
At the start: 4 copper layers, 0 parts

Commit message: Update sch and pcb
Parts:
- added C1: 16SEPF1000M, Capacitor_THT:CP_Radial_D10.0mm_P5.00mm, F.Cu at (84.7, 82.1)
- added C17: 0.1u, Capacitor_SMD:C_0603_1608Metric_Pad1.08x0.95mm_HandSolder, F.Cu at (70.2, 59.3)
- added C18: 0.1u, Capacitor_SMD:C_0603_1608Metric_Pad1.08x0.95mm_HandSolder, F.Cu at (92.1, 152.5)
- added C2: 16SKV100M6.3X5.5, Capacitor_SMD:CP_Elec_6.3x5.4, F.Cu at (131.2, 147.9)
- added C20: 0.1u, Capacitor_SMD:C_0603_1608Metric_Pad1.08x0.95mm_HandSolder, F.Cu at (165.6, 113.6)
- added C21: 0.1u, Capacitor_SMD:C_0603_1608Metric_Pad1.08x0.95mm_HandSolder, F.Cu at (70.2, 61.8)
- added C22: 1u, Capacitor_SMD:C_0603_1608Metric_Pad1.08x0.95mm_HandSolder, F.Cu at (70.2, 64.3)
- added C23: 1u, Capacitor_SMD:C_0603_1608Metric_Pad1.08x0.95mm_HandSolder, F.Cu at (70.2, 66.8)
- added C24: 0.1u, Capacitor_SMD:C_0603_1608Metric_Pad1.08x0.95mm_HandSolder, F.Cu at (70.2, 69.4)
- added C25: 0.1u, Capacitor_SMD:C_0603_1608Metric_Pad1.08x0.95mm_HandSolder, F.Cu at (70.2, 71.9)
- added C26: 0.1u, Capacitor_SMD:C_0603_1608Metric_Pad1.08x0.95mm_HandSolder, F.Cu at (70.2, 74.4)
- added C27: 0.1u, Capacitor_SMD:C_0603_1608Metric_Pad1.08x0.95mm_HandSolder, F.Cu at (70.2, 76.9)
- added C28: 0.1u, Capacitor_SMD:C_0603_1608Metric_Pad1.08x0.95mm_HandSolder, F.Cu at (74.6, 59.3)
- added C29: 0.1u, Capacitor_SMD:C_0603_1608Metric_Pad1.08x0.95mm_HandSolder, F.Cu at (74.6, 61.8)
- added C3: 16SKV100M6.3X5.5, Capacitor_SMD:CP_Elec_6.3x5.4, F.Cu at (131.2, 156.1)
- added C30: 0.1u, Capacitor_SMD:C_0603_1608Metric_Pad1.08x0.95mm_HandSolder, F.Cu at (74.6, 64.3)
- added C31: 0.1u, Capacitor_SMD:C_0603_1608Metric_Pad1.08x0.95mm_HandSolder, F.Cu at (74.6, 66.8)
- added C32: 0.1u, Capacitor_SMD:C_0603_1608Metric_Pad1.08x0.95mm_HandSolder, F.Cu at (74.6, 69.4)
- added C33: 0.1u, Capacitor_SMD:C_0603_1608Metric_Pad1.08x0.95mm_HandSolder, F.Cu at (74.6, 144.0)
- added C34: 0.1u, Capacitor_SMD:C_0603_1608Metric_Pad1.08x0.95mm_HandSolder, F.Cu at (123.7, 131.5)
- added C35: 1u, Capacitor_SMD:C_0603_1608Metric_Pad1.08x0.95mm_HandSolder, F.Cu at (165.6, 116.1)
- added C36: 0.1u, Capacitor_SMD:C_0603_1608Metric_Pad1.08x0.95mm_HandSolder, F.Cu at (123.7, 134.0)
- added C37: 0.1u, Capacitor_SMD:C_0603_1608Metric_Pad1.08x0.95mm_HandSolder, F.Cu at (123.7, 136.5)
- added C38: 0.1u, Capacitor_SMD:C_0603_1608Metric_Pad1.08x0.95mm_HandSolder, F.Cu at (123.7, 139.1)
- added C39: 2.2u, Capacitor_SMD:C_0603_1608Metric_Pad1.08x0.95mm_HandSolder, F.Cu at (195.1, 130.7)
- added C40: 2.2u, Capacitor_SMD:C_0603_1608Metric_Pad1.08x0.95mm_HandSolder, F.Cu at (195.1, 133.2)
- added C41: 0.1u, Capacitor_SMD:C_0603_1608Metric_Pad1.08x0.95mm_HandSolder, F.Cu at (195.1, 135.7)
- added C42: 0.1u, Capacitor_SMD:C_0603_1608Metric_Pad1.08x0.95mm_HandSolder, F.Cu at (195.1, 138.2)
- added C43: 0.1u, Capacitor_SMD:C_0603_1608Metric_Pad1.08x0.95mm_HandSolder, F.Cu at (195.1, 140.8)
- added C44: 0.1u, Capacitor_SMD:C_0603_1608Metric_Pad1.08x0.95mm_HandSolder, F.Cu at (199.4, 130.7)
- added C45: 0.1u, Capacitor_SMD:C_0603_1608Metric_Pad1.08x0.95mm_HandSolder, F.Cu at (199.4, 133.2)
- added C46: 4.7u, Capacitor_SMD:C_0805_2012Metric_Pad1.18x1.45mm_HandSolder, F.Cu at (188.2, 144.3)
- added C47: 0.1u, Capacitor_SMD:C_0603_1608Metric_Pad1.08x0.95mm_HandSolder, F.Cu at (199.4, 135.7)
- added C48: 1u, Capacitor_SMD:C_0603_1608Metric_Pad1.08x0.95mm_HandSolder, F.Cu at (199.4, 138.2)
- added C49: 0.1u, Capacitor_SMD:C_0603_1608Metric_Pad1.08x0.95mm_HandSolder, F.Cu at (92.1, 155.0)
- added C50: 0.1u, Capacitor_SMD:C_0603_1608Metric_Pad1.08x0.95mm_HandSolder, F.Cu at (92.1, 157.6)
- added C51: 0.1u, Capacitor_SMD:C_0603_1608Metric_Pad1.08x0.95mm_HandSolder, F.Cu at (92.1, 160.1)
- added C7: 4.7u, Capacitor_SMD:C_1210_3225Metric_Pad1.33x2.70mm_HandSolder, F.Cu at (101.1, 60.2)
- added C8: 4.7u, Capacitor_SMD:C_1210_3225Metric_Pad1.33x2.70mm_HandSolder, F.Cu at (101.1, 64.4)
- added C9: 3.3u, Capacitor_SMD:C_1210_3225Metric_Pad1.33x2.70mm_HandSolder, F.Cu at (101.1, 68.7)
- added D10: NUP2105L, Package_TO_SOT_SMD:SOT-23, F.Cu at (161.0, 114.6)
- added D11: SMBJ16CA(576-SMBJ16CA), Diode_SMD:D_SMB, F.Cu at (72.3, 92.3)
- added D13: MA10EB045, Diode_SMD:D_SOD-123, F.Cu at (181.1, 122.3)
- added D15: D_Schottky_Small, Diode_SMD:D_SOD-123, F.Cu at (84.0, 89.6)
- added D16: D_Schottky_Small, Diode_SMD:D_SOD-123, F.Cu at (84.0, 92.9)
- added F2: 1210L300SLWR, Fuse:Fuse_1210_3225Metric_Pad1.42x2.65mm_HandSolder, F.Cu at (97.3, 169.9)
- added FB1: MI0805K601R-10, Inductor_SMD:L_0805_2012Metric_Pad1.05x1.20mm_HandSolder, F.Cu at (109.9, 157.3)
- added FB3: 782639601, Inductor_SMD:L_0603_1608Metric_Pad1.05x0.95mm_HandSolder, F.Cu at (199.4, 140.8)
- added FL1: DLW32SH101XF2L, Unknown:FIL_DLW32SH101XF2L, F.Cu at (181.0, 114.5)
- added H1: MountingHole_Pad, MountingHole:MountingHole_3.2mm_M3_ISO7380_Pad, F.Cu at (97.2, 115.3)
- added H2: MountingHole_Pad, MountingHole:MountingHole_3.2mm_M3_ISO7380_Pad, F.Cu at (97.2, 122.5)
- added H3: MountingHole_Pad, MountingHole:MountingHole_3.2mm_M3_ISO7380_Pad, F.Cu at (97.2, 129.8)
- added H4: MountingHole_Pad, MountingHole:MountingHole_3.2mm_M3_ISO7380_Pad, F.Cu at (97.2, 137.0)
- added IC2: XC8114AA01PR-G, Unknown:XC6901D901PRG, F.Cu at (96.7, 80.5)
- added IC3: XC8114AA01PR-G, Unknown:XC6901D901PRG, F.Cu at (106.9, 165.5)
- added J1: 5077CR-16SMC2-BK-TR, Unknown:NELTRON_5077CR-16SMC2-BK-TR, F.Cu at (99.9, 154.3)
- added J10: Conn_01x06_Pin, Connector_JST:JST_XH_B6B-XH-A_1x06_P2.50mm_Vertical, F.Cu at (118.0, 114.3)
- added J12: Conn_01x03_Socket, Connector_JST:JST_XH_S3B-XH-A_1x03_P2.50mm_Horizontal, F.Cu at (201.1, 102.8)
- added J15: S2711-46R, pq_k_gentaro:S2711-46R, F.Cu at (67.4, 144.4)
- added J16: S2711-46R, pq_k_gentaro:S2711-46R, F.Cu at (67.4, 147.8)
- added J17: S2711-46R, pq_k_gentaro:S2711-46R, F.Cu at (67.4, 151.2)
- added J18: S2711-46R, pq_k_gentaro:S2711-46R, F.Cu at (67.4, 154.5)
- added J5: Conn_01x02_Socket, Connector_JST:JST_XH_S2B-XH-A_1x02_P2.50mm_Horizontal, F.Cu at (129.3, 133.6)
- added J6: Conn_01x02_Socket, Connector_JST:JST_VH_B2PS-VH_1x02_P3.96mm_Horizontal, F.Cu at (84.1, 60.4)
- added J7: Conn_01x02_Socket, Connector_JST:JST_XH_S2B-XH-A_1x02_P2.50mm_Horizontal, F.Cu at (138.8, 133.6)
- added J9: Conn_01x03_Socket, Connector_JST:JST_XH_S3B-XH-A_1x03_P2.50mm_Horizontal, F.Cu at (189.2, 102.8)
- added L1: BLM18PG471SN1D, Inductor_SMD:L_0603_1608Metric_Pad1.05x0.95mm_HandSolder, F.Cu at (74.6, 71.9)
- added Q1: TJ60S04M3L(T6L,1NQ, Package_TO_SOT_SMD:TO-252-2, F.Cu at (99.8, 89.1)
- added Q8: BSS138, Package_TO_SOT_SMD:SOT-23, F.Cu at (161.0, 119.0)
- added R1: 0, Resistor_SMD:R_0603_1608Metric_Pad0.98x0.95mm_HandSolder, F.Cu at (74.6, 74.4)
- added R10: 47k, Resistor_SMD:R_0603_1608Metric_Pad0.98x0.95mm_HandSolder, F.Cu at (123.7, 144.1)
- added R11: 47k, Resistor_SMD:R_0603_1608Metric_Pad0.98x0.95mm_HandSolder, F.Cu at (123.7, 146.6)
- added R12: 1k, Resistor_SMD:R_0603_1608Metric_Pad0.98x0.95mm_HandSolder, F.Cu at (123.7, 149.1)
- added R13: 10k, Resistor_SMD:R_0603_1608Metric_Pad0.98x0.95mm_HandSolder, F.Cu at (203.8, 130.7)
- added R14: 47k, Resistor_SMD:R_0603_1608Metric_Pad0.98x0.95mm_HandSolder, F.Cu at (203.8, 133.2)
- added R15: 10k, Resistor_SMD:R_0603_1608Metric_Pad0.98x0.95mm_HandSolder, F.Cu at (203.8, 135.7)
- added R16: 1k, Resistor_SMD:R_0603_1608Metric_Pad0.98x0.95mm_HandSolder, F.Cu at (92.1, 162.6)
- added R17: 5.1k, Resistor_SMD:R_0603_1608Metric_Pad0.98x0.95mm_HandSolder, F.Cu at (92.1, 165.1)
- added R18: 5.1k, Resistor_SMD:R_0603_1608Metric_Pad0.98x0.95mm_HandSolder, F.Cu at (92.1, 167.6)
- added R2: 100, Resistor_SMD:R_0603_1608Metric_Pad0.98x0.95mm_HandSolder, F.Cu at (74.6, 76.9)
- added R3: 47k, Resistor_SMD:R_0603_1608Metric_Pad0.98x0.95mm_HandSolder, F.Cu at (78.9, 59.3)
- added R34: 120, Resistor_SMD:R_0603_1608Metric_Pad0.98x0.95mm_HandSolder, F.Cu at (165.6, 118.6)
- added R4: 1k, Resistor_SMD:R_0603_1608Metric_Pad0.98x0.95mm_HandSolder, F.Cu at (78.9, 61.8)
- added R47: 1k, Resistor_SMD:R_0603_1608Metric, F.Cu at (180.5, 91.6)
- added R48: 47k, Resistor_SMD:R_0603_1608Metric, F.Cu at (180.5, 94.1)
- added R5: 47k, Resistor_SMD:R_0603_1608Metric_Pad0.98x0.95mm_HandSolder, F.Cu at (78.9, 64.3)
- added R6: 120, Resistor_SMD:R_0603_1608Metric_Pad0.98x0.95mm_HandSolder, F.Cu at (78.9, 66.8)
- added R7: 47k, Resistor_SMD:R_0603_1608Metric_Pad0.98x0.95mm_HandSolder, F.Cu at (78.9, 69.4)
- added R8: 1k, Resistor_SMD:R_0603_1608Metric_Pad0.98x0.95mm_HandSolder, F.Cu at (78.9, 71.9)
- added R9: 1k, Resistor_SMD:R_0603_1608Metric_Pad0.98x0.95mm_HandSolder, F.Cu at (123.7, 141.6)
- added S2: SS12SDP2, Unknown:SS12SDP2, F.Cu at (213.2, 103.5)
- added S3: SS12SDP2, Unknown:SS12SDP2, F.Cu at (94.6, 62.2)
- added S4: SS12SDP2, Unknown:SS12SDP2, F.Cu at (189.3, 133.6)
- added SW1: PTS645SK50SMTR92LFS, Unknown:SW4_PTS645SK50SMTR92LFS_CNK, F.Cu at (199.8, 147.3)
- added U1: LSM6DSK320XTR, Package_LGA:LGA-14_3x2.5mm_P0.5mm_LayoutBorder3x4y, F.Cu at (180.8, 118.6)
- added U10: ASGPDF254.A, Unknown:ASGPDF254.A, F.Cu at (171.1, 68.3)
- added U11: M78AR05-1/M78AR033-1, Unknown:M78AR05-1_M78AR033-1, F.Cu at (74.2, 88.8)
- added U12: UGCM1205XP, Unknown:UGCM1205XP, F.Cu at (165.7, 105.5)
- added U13: ADP151AUJZ-3.3, Package_TO_SOT_SMD:TSOT-23-5, F.Cu at (89.5, 90.3)
- added U14: BME280, Package_LGA:Bosch_LGA-8_2.5x2.5mm_P0.65mm_ClockwisePinNumbering, F.Cu at (78.7, 91.8)
- added U15: S01-30300500, Unknown:S01-30300500, F.Cu at (77.9, 125.9)
- added U16: FT230XS, Package_SO:SSOP-16_3.9x4.9mm_P0.635mm, F.Cu at (98.9, 164.6)
- added U17: USBLC6-2SC6, Package_TO_SOT_SMD:SOT-23-6, F.Cu at (110.0, 153.7)
- added U18: TCAN3414DR, Package_SO:SOIC-8_3.9x4.9mm_P1.27mm, F.Cu at (177.2, 87.1)
- added U19: USBLC6-4SC6, Package_TO_SOT_SMD:SOT-23-6, F.Cu at (117.7, 121.3)
- added U2: BMP585, Unknown:LGA9_BMP585_BOS-M, F.Cu at (175.7, 93.1)
- added U3: STM32H523RETx, Package_QFP:LQFP-64_10x10mm_P0.5mm, F.Cu at (165.8, 91.0)
- added U4: MAX-M10S, RF_GPS:ublox_MAX, F.Cu at (169.6, 130.1)
- added U5: E22-900T30D_E220-900T22S(JP)_versatile, Unknown:E22-900T30D_E220-900T22S(JP)_versatile, F.Cu at (263.8, 61.4)
- added U6: E22-900T30D_E220-900T22S(JP)_versatile, Unknown:E22-900T30D_E220-900T22S(JP)_versatile, F.Cu at (263.7, 35.8)
- added U7: MB85RS4MTYPF-G-BCERE1, Package_SO:SOIC-8_5.3x5.3mm_P1.27mm, F.Cu at (173.0, 115.9)
- added U8: TC7S14F, Package_TO_SOT_SMD:TSOT-23-5_HandSoldering, F.Cu at (152.9, 113.9)
- added U9: TC7S14F, Package_TO_SOT_SMD:TSOT-23-5_HandSoldering, F.Cu at (152.9, 118.5)
- added U9: TC7S14F, Package_TO_SOT_SMD:TSOT-23-5_HandSoldering, F.Cu at (140.0, 146.2)
Other:
- board outline added: 100 x 50 mm

Commit message: Add new parts
Parts:
- added C52: 0.1u, Capacitor_SMD:C_0603_1608Metric_Pad1.08x0.95mm_HandSolder, F.Cu at (166.8, 145.0)
- added C53: 0.1u, Capacitor_SMD:C_0603_1608Metric_Pad1.08x0.95mm_HandSolder, F.Cu at (166.8, 147.6)
- added U20: MB85RS4MTYPF-G-BCERE1, Package_SO:SOIC-8_5.3x5.3mm_P1.27mm, F.Cu at (159.4, 147.3)
- added U21: MB85RS4MTYPF-G-BCERE1, Package_SO:SOIC-8_5.3x5.3mm_P1.27mm, F.Cu at (159.4, 154.3)
Connections:
- net /~{FRAM_WP} renamed /~{FRAM1_WP}
- net /~{SPI4_CS} renamed /~{FRAM1_CS}
